File: RP_MD.sch (KiCad schematic (older format))
At the start: 23 parts, among them CN1 XT30PW-M, J2 Conn_01x04_Female, J3 Conn_01x04_Female, J4 Conn_01x06_Female, J5 Conn_01x06_Female, J6 Conn_01x04_Female, U10 NJM78L005, U9 MAX3458ED

Commit message: v1.1
Changed lines of the file:
@@
 P 2700 4900
 F 0 "J2" H 2728 4876 50  0000 L CNN
-F 1 "Conn_01x04_Female" H 2728 4785 50  0000 L CNN
+F 1 "Conn_01x04_Female" V 2650 5100 50  0000 L CNN
 F 2 "Connector_JST:JST_PH_B4B-PH-K_1x04_P2.00mm_Vertical" H 2700 4900 50  0001 C CNN
 F 3 "~" H 2700 4900 50  0001 C CNN

Commit message: kicad5
Parts:
- CN1: symbol maki_lib:XT30PW-M -> RP_MD-rescue:XT30PW-M-maki_lib
Changed lines of the file:
@@
 	1950 1350 1950 1250
 $Comp
-L maki_lib:XT30PW-M CN?
+L RP_MD-rescue:XT30PW-M-maki_lib CN?
 U 1 1 627A6CEC
 P 1700 2550
